File: kicad/verkotetut-sulat.sch (KiCad schematic (older format))
At the start: 1 part

Commit message: Make the initial connections in the schematic
Parts:
- removed U?: ESP-12E, symbol ESP-12E
- added C?: 33u, symbol C
- added P?: USB2Serial_connection, symbol CONN_01X06
- added R? (x2): 1k, symbol R
- added SW? (x2): SW_PUSH, symbol SW_PUSH
- added U?: ESP-12E, symbol ESP-12E
- added U?: LD1117S33TR, SOT-223, symbol LD1117S33TR
Connections:
- new net: R?.2, SW?.1, U?.1 (REST)
- new net: R?.2, SW?.1, U?.18 (GPIO0)
- new net +3V3: C?.1, P?.6 (P6), R?.1, R?.1, U?.17 (GPIO2), U?.2 (VO), U?.3 (CH_PD), U?.8 (VCC)
- new net +5V: P?.1 (P1), U?.3 (VI)
- new net ESP_ADC: U?.2 (ADC)
- new net ESP_CSO: U?.9 (CS0)
- new net ESP_MISO: U?.10 (MISO)
- new net ESP_MOSI: U?.13 (MOSI)
- new net ESP_RX: P?.3 (P3), U?.21 (RXD)
- new net ESP_SCLK: U?.14 (SCLK)
- new net ESP_TX: P?.4 (P4), U?.22 (TXD)
- new net GND: C?.2, P?.2 (P2), SW?.2, SW?.2, U?.1 (GND), U?.15 (GND), U?.16 (GPIO15)
- new net GPIO10: U?.12 (GPIO10)
- new net GPIO12: U?.6 (GPIO12)
- new net GPIO13: U?.7 (GPIO13)
- new net GPIO14: U?.5 (GPIO14)
- new net GPIO16: U?.4 (GPIO16)
- new net GPIO4: U?.19 (GPIO4)
- new net GPIO5: U?.20 (GPIO5)
- new net GPIO9: U?.11 (GPIO9)
- new net USB2Serial_DTR: P?.5 (P5)

Commit message: Finish schematic
Parts:
- removed U?: LD1117S33TR, SOT-223, symbol LD1117S33TR
- added C?: 33u, symbol C
- added D?: LED, symbol LED
- added P?: Battery connection, symbol CONN_01X02
- added P?: GPIO, symbol CONN_01X08
- added P?: Programming pins, symbol CONN_01X04
- added R?: 145, symbol R
- added R?: 240, symbol R
- added R?: 330, symbol R
- added U?: LM317T, TO-220, symbol LM317T
Connections:
- net +3V3: now also C?.1, D?.2 (A), R?.1, U?.2 (OUT)
- net ESP_CSO: now also P?.4 (P4)
- net ESP_MISO: now also P?.3 (P3)
- net ESP_MOSI: now also P?.2 (P2)
- net ESP_SCLK: now also P?.1 (P1)
- net GND: now also C?.2, P?.2 (P2), R?.2, R?.2
- net GPIO10: now also P?.4 (P4)
- net GPIO12: now also P?.5 (P5)
- net GPIO13: now also P?.6 (P6)
- net GPIO14: now also P?.7 (P7)
- net GPIO16: now also P?.8 (P8)
- net GPIO4: now also P?.1 (P1)
- net GPIO5: now also P?.2 (P2)
- net GPIO9: now also P?.3 (P3)
- new net: R?.1, R?.2, U?.1 (ADJ)
- new net: D?.1 (K), R?.1
- new net +9V: P?.1 (P1), U?.3 (IN)
Other:
- note added: "The circuit assumes\na voltage of 9V, but\nanything from 6.5V\nto 20V should be okay."
- moved on the sheet: P?

Commit message: Add a LED to GPIO4 and a pinout for ADC
Parts:
- removed P?: GPIO, symbol CONN_01X08
- added D?: LED, symbol LED
- added P?: GPIO and ADC, symbol CONN_01X09
- added R?: 330, symbol R
- R?: value 145 -> 150
Connections:
- net ESP_ADC: now also P?.9 (P9)
- net GND: now also R?.2
- net GPIO10: now also P?.4 (P4)
- net GPIO12: now also P?.5 (P5)
- net GPIO13: now also P?.6 (P6)
- net GPIO14: now also P?.7 (P7)
- net GPIO16: now also P?.8 (P8)
- net GPIO4: now also D?.2 (A), P?.1 (P1)
- net GPIO5: now also P?.2 (P2)
- net GPIO9: now also P?.3 (P3)
- new net: D?.1 (K), R?.1
Changed lines of the file:
@@
 P 8750 1250
 F 0 "R?" V 8830 1250 50  0000 C CNN
-F 1 "145" V 8750 1250 50  0000 C CNN
+F 1 "150" V 8750 1250 50  0000 C CNN
 F 2 "" V 8680 1250 50  0000 C CNN
 F 3 "" H 8750 1250 50  0000 C CNN
@@
 Wire Wire Line
 	10200 1850 10200 2000
-$Comp
-L CONN_01X08 P?
-U 1 1 582B26F4
-P 2100 1900
-F 0 "P?" H 2100 2350 50  0000 C CNN
-F 1 "GPIO" V 2200 1900 50  0000 C CNN
-F 2 "" H 2100 1900 50  0000 C CNN
-F 3 "" H 2100 1900 50  0000 C CNN
-	1    2100 1900
-	-1   0    0    1
-$EndComp
 Text GLabel 2450 2250 2    60   BiDi ~ 0
 GPIO4
@@
 Wire Wire Line
 	2750 5150 2550 5150
+$Comp
+L CONN_01X09 P?
+U 1 1 582B382C
+P 2100 1850
+F 0 "P?" H 2100 2350 50  0000 C CNN
+F 1 "GPIO and ADC" V 2200 1850 50  0000 C CNN
+F 2 "" H 2100 1850 50  0000 C CNN
+F 3 "" H 2100 1850 50  0000 C CNN
+	1    2100 1850
+	-1   0    0    1
+$EndComp
+Text GLabel 2450 1450 2    60   Output ~ 0
+ESP_ADC
+Wire Wire Line
+	2450 1450 2300 1450
+$Comp
+L LED D?
+U 1 1 582B3E8B
+P 2350 2600
+F 0 "D?" H 2350 2700 50  0000 C CNN
+F 1 "LED" H 2350 2500 50  0000 C CNN
+F 2 "" H 2350 2600 50  0000 C CNN
+F 3 "" H 2350 2600 50  0000 C CNN
+	1    2350 2600
+	0    -1   -1   0
+$EndComp
+$Comp
+L R R?
+U 1 1 582B3E92
+P 2350 3050
+F 0 "R?" V 2430 3050 50  0000 C CNN
+F 1 "330" V 2350 3050 50  0000 C CNN
+F 2 "" V 2280 3050 50  0000 C CNN
+F 3 "" H 2350 3050 50  0000 C CNN
+	1    2350 3050
+	1    0    0    -1
+$EndComp
+$Comp
+L GND #PWR?
+U 1 1 582B3E98
+P 2350 3350
+F 0 "#PWR?" H 2350 3100 50  0001 C CNN
+F 1 "GND" H 2350 3200 50  0000 C CNN
+F 2 "" H 2350 3350 50  0000 C CNN
+F 3 "" H 2350 3350 50  0000 C CNN
+	1    2350 3350
+	1    0    0    -1
+$EndComp
+Wire Wire Line
+	2350 2800 2350 2900
+Wire Wire Line
+	2350 3200 2350 3350
+Wire Wire Line
+	2350 2400 2350 2250
+Connection ~ 2350 2250
 $EndSCHEMATC

Commit message: Create netlist
Parts:
- added C102: 0.1u, symbol C
- C103: renamed from C?; value 33u -> 1u
- gave numbers to parts that had none: 17
Connections:
- net +9V: now also C102.1
- net GND: now also C102.2

Commit message: Start PCB design
Parts:
- removed C101: 33u, symbol C
- removed C102: 0.1u, symbol C
- removed C103: 1u, symbol C
- removed SW102: SW_PUSH, symbol SW_PUSH
- added C101: 33u, Capacitors_ThroughHole:C_Radial_D10_L21_P5, symbol CP1
- added C102, C103: 1u, Capacitors_ThroughHole:C_Radial_D5_L11_P2, symbol CP1
- added SW102: SPST, nikulaj-kicad:SPDT_SMD_SIDE, symbol SPST
- D101, D102: footprint (none) -> LEDs:LED_0603
- P101: footprint (none) -> Pin_Headers:Pin_Header_Straight_1x09
- P102: footprint (none) -> Pin_Headers:Pin_Header_Straight_1x04
- P103: footprint (none) -> Pin_Headers:Pin_Header_Straight_1x02
- P104: footprint (none) -> Pin_Headers:Pin_Header_Straight_1x06
- R101, R102, R103, R106: footprint (none) -> Resistors_SMD:R_0603
- R104, R105: footprint (none) -> Resistors_SMD:R_0805
- SW101: footprint (none) -> Buttons_Switches_SMD:SW_SPST_B3S-1000
- U101: footprint (none) -> nikulaj-kicad:ESP-12E
- U102: footprint TO-220 -> TO_SOT_Packages_THT:TO-220_Neutral123_Horizontal
Connections:
- net +3V3: now also C101.1, C103.1
- net +9V: now also C102.1
- net GND: now also C101.2, C102.2, C103.2, SW102.2
- net at R103.2, U101.18 (GPIO0): now also SW102.1
Other:
- moved on the sheet: D102, P104, R104, R105, R106, U102
