File: kicad/verkotetut-sulat.kicad_pcb (KiCad board)
At the start: 2 copper layers, 19 parts, among them P101 GPIO and ADC, P102 Programming pins, P103 Battery connection, P104 USB2Serial_connection, SW101 SW_PUSH, SW102 SPST, U101 ESP-12E, U102 LM317T

Commit message: Work on pcb
Parts:
- D101, D102, R101, R102, R103, R104, R105, R106, SW101, SW102, U101: moved to B.Cu
- moved SW102 88.6 mm to (134.6, 72.4), turned to 180 degrees
- moved R104 85.4 mm to (129.5, 106.7), turned to 180 degrees
- moved C103 85.0 mm to (134.0, 109.2), turned to 270 degrees
- moved P104 85.0 mm to (118.1, 94.0), turned to 180 degrees
- moved R103 84.9 mm to (134.6, 79.4)
- moved P102 70.6 mm to (118.1, 101.0)
- moved C102 69.5 mm to (142.9, 117.5), turned to 270 degrees
- moved R105 64.3 mm to (128.3, 110.5), turned to 270 degrees
- moved P103 63.1 mm to (154.9, 117.5)
- moved R102 61.9 mm to (163.8, 82.5), turned to 90 degrees
- moved SW101 59.5 mm to (170.8, 78.1), turned to 180 degrees
- moved C101 52.3 mm to (134.6, 90.8), turned to 270 degrees
- moved D102 50.9 mm to (170.2, 106.0), turned to 90 degrees
- moved D101 45.3 mm to (173.4, 106.0), turned to 90 degrees
- moved R101 42.8 mm to (173.4, 109.2), turned to 270 degrees
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Routing:
- net GND: track 0.00 -> 150.0 mm, vias 0 -> 2
- net +3V3: track 0.00 -> 117.6 mm
- net ESP_CSO: track 0.00 -> 46.3 mm
- net ESP_MISO: track 0.00 -> 43.7 mm
- net GPIO10: track 0.00 -> 40.2 mm, vias 0 -> 2
- net ESP_MOSI: track 0.00 -> 36.1 mm
- net GPIO9: track 0.00 -> 34.0 mm, vias 0 -> 2
- net ESP_ADC: track 0.00 -> 33.0 mm
- net ESP_SCLK: track 0.00 -> 32.3 mm
- net ESP_RX: track 0.00 -> 29.9 mm
- net ESP_TX: track 0.00 -> 29.6 mm
- net Net-(R103-Pad2): track 0.00 -> 28.0 mm
- net GPIO13: track 0.00 -> 24.1 mm, vias 0 -> 2
- net GPIO16: track 0.00 -> 23.7 mm
- net GPIO14: track 0.00 -> 23.5 mm
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Other:
- board outline added: 73.7 x 55.9 mm
- net class Default: clearance 0.2 -> 0.3; trace_width 0.25 -> 0.3
- rule trace_clearance: 0.2 -> 0.3

Commit message: Draw all connections
Routing:
- net GND: track 150.0 -> 221.3 mm
- net GPIO4: track 10.4 -> 60.1 mm, vias 0 -> 2
- net GPIO5: track 0.00 -> 48.2 mm, vias 0 -> 2
- net +3V3: track 117.6 -> 133.2 mm, vias 0 -> 2
- net GPIO9: track 34.0 -> 33.0 mm
Changed lines of the file:
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@@
   (general
     (links 49)
-    (no_connects 5)
-    (area 92.9288 71.669999 189.955479 134.530001)
+    (no_connects 0)
+    (area 112.319999 70.409999 186.130001 126.440001)
     (thickness 1.6)
     (drawings 4)
-    (tracks 149)
+    (tracks 183)
     (zones 0)
     (modules 19)
@@
     (add_net USB2Serial_DTR)
   )
+  (module TO_SOT_Packages_THT:TO-220_Neutral123_Horizontal (layer F.Cu)
+    (at 142.875 109.22 270)
+    (descr "TO-220, Neutral, Horizontal,")
+    (tags "TO-220, Neutral, Horizontal,")
+    (fp_text reference U102 (at 0 -22.3012 270) (layer F.SilkS)
+      (effects (font (size 1 1) (thickness 0.15)))
+    )
+    (fp_text value LM317T (at -0.29972 3.44932 270) (layer F.Fab)
+      (effects (font (size 1 1) (thickness 0.15)))
+    )
+    (fp_circle (center 0 -16.764) (end 1.778 -14.986) (layer F.SilkS) (width 0.15))
+    (fp_line (start -2.54 -3.683) (end -2.54 -1.905) (layer F.SilkS) (width 0.15))
+    (fp_line (start 0 -3.683) (end 0 -1.905) (layer F.SilkS) (width 0.15))
+    (fp_line (start 2.54 -3.683) (end 2.54 -1.905) (layer F.SilkS) (width 0.15))
+    (fp_line (start 5.334 -12.192) (end 5.334 -20.193) (layer F.SilkS) (width 0.15))
+    (fp_line (start 5.334 -20.193) (end -5.334 -20.193) (layer F.SilkS) (width 0.15))
+    (fp_line (start -5.334 -20.193) (end -5.334 -12.192) (layer F.SilkS) (width 0.15))
+    (fp_line (start 5.334 -3.683) (end 5.334 -12.192) (layer F.SilkS) (width 0.15))
+    (fp_line (start 5.334 -12.192) (end -5.334 -12.192) (layer F.SilkS) (width 0.15))
+    (fp_line (start -5.334 -12.192) (end -5.334 -3.683) (layer F.SilkS) (width 0.15))
+    (fp_line (start 0 -3.683) (end -5.334 -3.683) (layer F.SilkS) (width 0.15))
+    (fp_line (start 0 -3.683) (end 5.334 -3.683) (layer F.SilkS) (width 0.15))
+    (pad 2 thru_hole oval (at 0 0) (size 2.49936 1.50114) (drill 1.00076) (layers *.Cu *.Mask)
+      (net 1 +3V3))
+    (pad 1 thru_hole oval (at -2.54 0) (size 2.49936 1.50114) (drill 1.00076) (layers *.Cu *.Mask)
+      (net 25 "Net-(R104-Pad2)"))
+    (pad 3 thru_hole oval (at 2.54 0) (size 2.49936 1.50114) (drill 1.00076) (layers *.Cu *.Mask)
+      (net 3 +9V))
+    (pad "" np_thru_hole circle (at 0 -16.764) (size 3.79984 3.79984) (drill 3.79984) (layers *.Cu *.Mask))
+    (model TO_SOT_Packages_THT.3dshapes/TO-220_Neutral123_Horizontal.wrl
+      (at (xyz 0 0 0))
+      (scale (xyz 0.3937 0.3937 0.3937))
+      (rotate (xyz 0 0 0))
+    )
+  )
   (module Capacitors_ThroughHole:C_Radial_D10_L21_P5 (layer F.Cu)
     (at 134.62 90.805 270)
@@
     )
   )
-  (module TO_SOT_Packages_THT:TO-220_Neutral123_Horizontal (layer F.Cu)
-    (at 142.875 109.22 270)
-    (descr "TO-220, Neutral, Horizontal,")
-    (tags "TO-220, Neutral, Horizontal,")
-    (fp_text reference U102 (at 0 -22.3012 270) (layer F.SilkS)
-      (effects (font (size 1 1) (thickness 0.15)))
-    )
-    (fp_text value LM317T (at -0.29972 3.44932 270) (layer F.Fab)
-      (effects (font (size 1 1) (thickness 0.15)))
-    )
-    (fp_circle (center 0 -16.764) (end 1.778 -14.986) (layer F.SilkS) (width 0.15))
-    (fp_line (start -2.54 -3.683) (end -2.54 -1.905) (layer F.SilkS) (width 0.15))
-    (fp_line (start 0 -3.683) (end 0 -1.905) (layer F.SilkS) (width 0.15))
-    (fp_line (start 2.54 -3.683) (end 2.54 -1.905) (layer F.SilkS) (width 0.15))
-    (fp_line (start 5.334 -12.192) (end 5.334 -20.193) (layer F.SilkS) (width 0.15))
-    (fp_line (start 5.334 -20.193) (end -5.334 -20.193) (layer F.SilkS) (width 0.15))
-    (fp_line (start -5.334 -20.193) (end -5.334 -12.192) (layer F.SilkS) (width 0.15))
-    (fp_line (start 5.334 -3.683) (end 5.334 -12.192) (layer F.SilkS) (width 0.15))
-    (fp_line (start 5.334 -12.192) (end -5.334 -12.192) (layer F.SilkS) (width 0.15))
-    (fp_line (start -5.334 -12.192) (end -5.334 -3.683) (layer F.SilkS) (width 0.15))
-    (fp_line (start 0 -3.683) (end -5.334 -3.683) (layer F.SilkS) (width 0.15))
-    (fp_line (start 0 -3.683) (end 5.334 -3.683) (layer F.SilkS) (width 0.15))
-    (pad 2 thru_hole oval (at 0 0) (size 2.49936 1.50114) (drill 1.00076) (layers *.Cu *.Mask)
-      (net 1 +3V3))
-    (pad 1 thru_hole oval (at -2.54 0) (size 2.49936 1.50114) (drill 1.00076) (layers *.Cu *.Mask)
-      (net 25 "Net-(R104-Pad2)"))
-    (pad 3 thru_hole oval (at 2.54 0) (size 2.49936 1.50114) (drill 1.00076) (layers *.Cu *.Mask)
-      (net 3 +9V))
-    (pad "" np_thru_hole circle (at 0 -16.764) (size 3.79984 3.79984) (drill 3.79984) (layers *.Cu *.Mask))
-    (model TO_SOT_Packages_THT.3dshapes/TO-220_Neutral123_Horizontal.wrl
-      (at (xyz 0 0 0))
-      (scale (xyz 0.3937 0.3937 0.3937))
-      (rotate (xyz 0 0 0))
-    )
-  )
   (gr_line (start 112.395 126.365) (end 112.395 70.485) (angle 90) (layer Edge.Cuts) (width 0.15))
   (gr_line (start 186.055 126.365) (end 112.395 126.365) (angle 90) (layer Edge.Cuts) (width 0.15))
   (gr_line (start 186.055 70.485) (end 186.055 126.365) (angle 90) (layer Edge.Cuts) (width 0.15))
   (gr_line (start 112.395 70.485) (end 186.055 70.485) (angle 90) (layer Edge.Cuts) (width 0.15))
+  (segment (start 133.87 79.375) (end 133.87 83.705) (width 0.3) (layer B.Cu) (net 1))
+  (segment (start 135.89 90.805) (end 134.62 90.805) (width 0.3) (layer B.Cu) (net 1))
+  (segment (start 138.43 88.265) (end 135.89 90.805) (width 0.3) (layer B.Cu) (net 1))
+  (via (at 138.43 88.265) (size 0.6) (drill 0.4) (layers F.Cu B.Cu) (net 1))
+  (segment (start 133.985 83.82) (end 138.43 88.265) (width 0.3) (layer F.Cu) (net 1))
+  (via (at 133.985 83.82) (size 0.6) (drill 0.4) (layers F.Cu B.Cu) (net 1))
+  (segment (start 133.87 83.705) (end 133.985 83.82) (width 0.3) (layer B.Cu) (net 1))
   (segment (start 142.875 109.22) (end 151.765 109.22) (width 0.3) (layer B.Cu) (net 1))
   (segment (start 155.6893 105.2957) (end 170.18 105.2957) (width 0.3) (layer B.Cu) (net 1))
@@
   (segment (start 159.385 84.645) (end 162.485 84.645) (width 0.3) (layer B.Cu) (net 1))
   (segment (start 162.485 84.645) (end 163.83 83.3) (width 0.3) (layer B.Cu) (net 1))
+  (segment (start 134.62 76.39) (end 134.62 76.835) (width 0.3) (layer B.Cu) (net 2))
+  (segment (start 114.3 91.44) (end 115.2525 92.3925) (width 0.3) (layer B.Cu) (net 2))
+  (segment (start 114.3 78.74) (end 114.3 91.44) (width 0.3) (layer B.Cu) (net 2))
+  (segment (start 115.57 77.47) (end 114.3 78.74) (width 0.3) (layer B.Cu) (net 2))
+  (segment (start 133.985 77.47) (end 115.57 77.47) (width 0.3) (layer B.Cu) (net 2))
+  (segment (start 134.62 76.835) (end 133.985 77.47) (width 0.3) (layer B.Cu) (net 2))
+  (segment (start 128.27 111.44) (end 115.885 111.44) (width 0.3) (layer B.Cu) (net 2))
+  (segment (start 116.205 91.44) (end 118.11 91.44) (width 0.3) (layer B.Cu) (net 2))
+  (segment (start 114.3 93.345) (end 115.2525 92.3925) (width 0.3) (layer B.Cu) (net 2))
+  (segment (start 115.2525 92.3925) (end 116.205 91.44) (width 0.3) (layer B.Cu) (net 2))
+  (segment (start 114.3 109.855) (end 114.3 93.345) (width 0.3) (layer B.Cu) (net 2))
+  (segment (start 115.885 111.44) (end 114.3 109.855) (width 0.3) (layer B.Cu) (net 2))
   (segment (start 128.27 111.44) (end 133.765 111.44) (width 0.3) (layer B.Cu) (net 2))
   (segment (start 133.765 111.44) (end 133.985 111.22) (width 0.3) (layer B.Cu) (net 2))
@@
   (segment (start 142.875 111.76) (end 142.875 117.475) (width 0.3) (layer B.Cu) (net 3))
   (segment (start 154.94 117.475) (end 142.875 117.475) (width 0.3) (layer B.Cu) (net 3))
+  (segment (start 145.385 86.645) (end 141.955 86.645) (width 0.3) (layer B.Cu) (net 4))
+  (segment (start 177.165 97.79) (end 180.34 97.79) (width 0.3) (layer B.Cu) (net 4))
+  (segment (start 175.895 96.52) (end 177.165 97.79) (width 0.3) (layer B.Cu) (net 4))
+  (via (at 175.895 96.52) (size 0.6) (drill 0.4) (layers F.Cu B.Cu) (net 4))
+  (segment (start 148.59 96.52) (end 175.895 96.52) (width 0.3) (layer F.Cu) (net 4))
+  (segment (start 140.335 88.265) (end 148.59 96.52) (width 0.3) (layer F.Cu) (net 4))
+  (via (at 140.335 88.265) (size 0.6) (drill 0.4) (layers F.Cu B.Cu) (net 4))
+  (segment (start 141.955 86.645) (end 140.335 88.265) (width 0.3) (layer B.Cu) (net 4))
   (segment (start 173.355 105.2957) (end 173.355 104.775) (width 0.3) (layer B.Cu) (net 4))
   (segment (start 173.355 104.775) (end 180.34 97.79) (width 0.3) (layer B.Cu) (net 4))
   (segment (start 173.355 106.7943) (end 173.355 108.47) (width 0.3) (layer B.Cu) (net 5))
   (segment (start 170.18 106.7943) (end 170.18 108.47) (width 0.3) (layer B.Cu) (net 6))
+  (segment (start 145.385 84.645) (end 142.05 84.645) (width 0.3) (layer B.Cu) (net 7))
+  (segment (start 177.165 95.25) (end 180.34 95.25) (width 0.3) (layer B.Cu) (net 7))
+  (via (at 177.165 95.25) (size 0.6) (drill 0.4) (layers F.Cu B.Cu) (net 7))
+  (segment (start 150.495 95.25) (end 177.165 95.25) (width 0.3) (layer F.Cu) (net 7))
+  (segment (start 140.97 85.725) (end 150.495 95.25) (width 0.3) (layer F.Cu) (net 7))
+  (via (at 140.97 85.725) (size 0.6) (drill 0.4) (layers F.Cu B.Cu) (net 7))
+  (segment (start 142.05 84.645) (end 140.97 85.725) (width 0.3) (layer B.Cu) (net 7))
+  (segment (start 170.18 97.79) (end 172.72 97.79) (width 0.3) (layer F.Cu) (net 8))
+  (via (at 172.72 97.79) (size 0.6) (drill 0.4) (layers F.Cu B.Cu) (net 8))
   (segment (start 153.395 96.395) (end 153.395 99.42) (width 0.3) (layer B.Cu) (net 8))
   (segment (start 177.8 92.71) (end 180.34 92.71) (width 0.3) (layer B.Cu) (net 8))
-  (segment (start 171.45 99.06) (end 177.8 92.71) (width 0.3) (layer B.Cu) (net 8))
-  (via (at 171.45 99.06) (size 0.6) (drill 0.4) (layers F.Cu B.Cu) (net 8))
-  (segment (start 170.18 97.79) (end 171.45 99.06) (width 0.3) (layer F.Cu) (net 8))
+  (segment (start 172.72 97.79) (end 177.8 92.71) (width 0.3) (layer B.Cu) (net 8))
   (segment (start 168.275 97.79) (end 170.18 97.79) (width 0.3) (layer F.Cu) (net 8))
   (segment (start 166.37 99.695) (end 168.275 97.79) (width 0.3) (layer F.Cu) (net 8))

Commit message: Pour copper
Routing:
- added copper zone on B.Cu, net GND
- added copper zone on F.Cu, net GND
Other:
- rule trace_min: 0.2 -> 0.3
Changed lines of the file:
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@@
     (links 49)
     (no_connects 0)
-    (area 112.319999 70.409999 186.130001 126.440001)
+    (area 109.214761 62.315 186.130001 126.440001)
     (thickness 1.6)
     (drawings 4)
@@
     (trace_clearance 0.3)
     (zone_clearance 0.508)
-    (zone_45_only no)
-    (trace_min 0.2)
+    (zone_45_only yes)
+    (trace_min 0.3)
     (segment_width 0.2)
     (edge_width 0.15)
@@
   (segment (start 128.59 106.68) (end 128.59 109.22) (width 0.3) (layer B.Cu) (net 25))
   (segment (start 128.59 109.22) (end 128.27 109.54) (width 0.3) (layer B.Cu) (net 25))
+  (zone (net 2) (net_name GND) (layer F.Cu) (hatch edge 0.508)
+    (connect_pads (clearance 0.508))
+    (min_thickness 0.254)
+    (fill yes (arc_segments 16) (thermal_gap 0.508) (thermal_bridge_width 0.508))
+    (polygon
+      (pts
+        (xy 186.055 126.365) (xy 112.395 126.365) (xy 112.395 70.485) (xy 186.055 70.485)
+      )
+    )
+  )
+  (zone (net 2) (net_name GND) (layer B.Cu) (hatch edge 0.508)
+    (connect_pads (clearance 0.508))
+    (min_thickness 0.254)
+    (fill yes (arc_segments 16) (thermal_gap 0.508) (thermal_bridge_width 0.508))
+    (polygon
+      (pts
+        (xy 186.055 126.365) (xy 112.395 126.365) (xy 112.395 70.485) (xy 186.055 70.485)
+      )
+    )
+  )
+  (zone (net 0) (net_name "") (layer B.Cu) (hatch edge 0.508)
+    (connect_pads (clearance 0.508))
+    (min_thickness 0.254)
+    (keepout (tracks not_allowed) (vias not_allowed) (copperpour not_allowed))
+    (fill (arc_segments 16) (thermal_gap 0.508) (thermal_bridge_width 0.508))
+    (polygon
+      (pts
+        (xy 161.925 78.105) (xy 142.875 78.105) (xy 142.875 71.12) (xy 161.925 71.12)
+      )
+    )
+  )
+  (zone (net 0) (net_name "") (layer F.Cu) (hatch edge 0.508)
+    (connect_pads (clearance 0.508))
+    (min_thickness 0.254)
+    (keepout (tracks not_allowed) (vias not_allowed) (copperpour not_allowed))
+    (fill (arc_segments 16) (thermal_gap 0.508) (thermal_bridge_width 0.508))
+    (polygon
+      (pts
+        (xy 161.925 78.105) (xy 142.875 78.105) (xy 142.875 71.12) (xy 161.925 71.12)
+      )
+    )
+  )
 )
